Commit message: fix(mpd): align bimanual kinematics and constraints

File: mpd/torch_robotics/torch_robotics/data/urdf/robots/marvin/marvin_bimanual_mpd.urdf (robot description, URDF)
Before this commit: robot marvin_bimanual_mpd, 17 links, 16 joints
Joints:
- joint Joint2_L: origin xyz=0 0 0.12 rpy=0 1.570796 0 -> xyz=0.12 0 0 rpy=0 0 0
- joint Joint2_R: origin xyz=0 0 0.12 rpy=0 1.570796 0 -> xyz=0.12 0 0 rpy=0 0 0
- joint Joint4_L: origin xyz=0.25 0 0 rpy=0 1.570796 0 -> xyz=0.25 0 0 rpy=0 0 0
- joint Joint4_R: origin xyz=0.25 0 0 rpy=0 1.570796 0 -> xyz=0.25 0 0 rpy=0 0 0
- joint Joint6_L: origin xyz=0.18 0 0 rpy=0 1.570796 0 -> xyz=0.18 0 0 rpy=0 0 0
- joint Joint6_R: origin xyz=0.18 0 0 rpy=0 1.570796 0 -> xyz=0.18 0 0 rpy=0 0 0

Commit message: feat(mpd): migrate Marvin bimanual geometry assets

File: mpd/torch_robotics/torch_robotics/data/urdf/robots/marvin/marvin_bimanual_mpd.urdf (robot description, URDF)
Before this commit: robot marvin_bimanual_mpd, 17 links, 16 joints
Links:
- removed link base_L
- removed link base_R
- removed link link1_L
- removed link link1_R
- removed link link2_L
- removed link link2_R
- removed link link3_L
- removed link link3_R
- removed link link4_L
- removed link link4_R
- removed link link5_L
- removed link link5_R
- removed link link6_L
- removed link link6_R
- added link Base_L, mass 1.1962; collision mesh filename=meshes/m6/Base_L.STL; visual mesh filename=meshes/m6/Base_L.STL
- added link Base_R, mass 1.1962; collision mesh filename=meshes/m6/Base_R.STL; visual mesh filename=meshes/m6/Base_R.STL
- added link Link1_L, mass 1.9705; collision mesh filename=meshes/m6/Link1_L.STL; visual mesh filename=meshes/m6/Link1_L.STL
- added link Link1_R, mass 1.9705; collision mesh filename=meshes/m6/Link1_R.STL; visual mesh filename=meshes/m6/Link1_R.STL
- added link Link2_L, mass 2.24398; collision mesh filename=meshes/m6/Link2_L.STL; visual mesh filename=meshes/m6/Link2_L.STL
- added link Link2_R, mass 2.24398; collision mesh filename=meshes/m6/Link2_R.STL; visual mesh filename=meshes/m6/Link2_R.STL
- added link Link3_L, mass 1.9242; collision mesh filename=meshes/m6/Link3_L.STL; visual mesh filename=meshes/m6/Link3_L.STL
- added link Link3_R, mass 1.9242; collision mesh filename=meshes/m6/Link3_R.STL; visual mesh filename=meshes/m6/Link3_R.STL
- added link Link4_L, mass 1.6085; collision mesh filename=meshes/m6/Link4_L.STL; visual mesh filename=meshes/m6/Link4_L.STL
- added link Link4_R, mass 1.6085; collision mesh filename=meshes/m6/Link4_R.STL; visual mesh filename=meshes/m6/Link4_R.STL
- added link Link5_L, mass 2.0883; collision mesh filename=meshes/m6/Link5_L.STL; visual mesh filename=meshes/m6/Link5_L.STL
- added link Link5_R, mass 2.0883; collision mesh filename=meshes/m6/Link5_R.STL; visual mesh filename=meshes/m6/Link5_R.STL
- added link Link6_L, mass 0.72496; collision mesh filename=meshes/m6/Link6_L.STL; visual mesh filename=meshes/m6/Link6_L.STL
- added link Link6_R, mass 0.72496; collision mesh filename=meshes/m6/Link6_R.STL; visual mesh filename=meshes/m6/Link6_R.STL
- added link Link7_L, mass 0.68606; collision mesh filename=meshes/m6/Link7_L.STL; visual mesh filename=meshes/m6/Link7_L.STL
- added link Link7_R, mass 0.68606; collision mesh filename=meshes/m6/Link7_R.STL; visual mesh filename=meshes/m6/Link7_R.STL
- added link column_link; collision cylinder length=1.0 radius=0.06; visual cylinder length=1.0 radius=0.06
- added link tracking_base_link
- added link world
- link base_link: mass None -> 1.21; geometry collision mesh filename=meshes/base/base_link.STL; visual mesh filename=meshes/base/base_link.STL
Joints:
- removed joint mount_L
- removed joint mount_R
- added joint base_mount_joint: type fixed, parent world, child base_link, origin xyz=0 0 0 rpy=0 0 0
- added joint base_to_column: type fixed, parent base_link, child column_link, origin xyz=0 0 -0.50 rpy=0 0 0
- added joint base_to_left_arm: type fixed, parent base_link, child Base_L, origin xyz=0 0.026 0.070 rpy=-1.57 0 0
- added joint base_to_right_arm: type fixed, parent base_link, child Base_R, origin xyz=0 -0.026 0.070 rpy=1.57 0 0
- added joint base_to_tracking_base: type fixed, parent base_link, child tracking_base_link, origin xyz=0 0 -1 rpy=0 0 0
- added joint joint_flange_L: type fixed, parent Link7_L, child flange_L, origin xyz=0 -0.095 0 rpy=1.5708 -1.5708 0
- added joint joint_flange_R: type fixed, parent Link7_R, child flange_R, origin xyz=0 -0.095 0 rpy=1.5708 -1.5708 0
- joint Joint1_L: child link1_L -> Link1_L; limit lower=-3.14159 upper=3.14159 effort=100 velocity=2 -> lower=-2.9671 upper=2.9671 effort=108.0 velocity=3.1416; origin xyz=0 0 0 rpy=0 0 0 -> xyz=0 0 0.1745 rpy=0 0 0; parent base_L -> Base_L
- joint Joint1_R: child link1_R -> Link1_R; limit lower=-3.14159 upper=3.14159 effort=100 velocity=2 -> lower=-2.9671 upper=2.9671 effort=108.0 velocity=3.1416; origin xyz=0 0 0 rpy=0 0 0 -> xyz=0 0 0.1745 rpy=0 0 0; parent base_R -> Base_R
- joint Joint2_L: child link2_L -> Link2_L; limit lower=-2.6 upper=2.6 effort=100 velocity=2 -> lower=-2.0944 upper=2.0944 effort=108.0 velocity=3.1416; origin xyz=0.12 0 0 rpy=0 0 0 -> xyz=0 0 0 rpy=1.5708 0 0; parent link1_L -> Link1_L
- joint Joint2_R: child link2_R -> Link2_R; limit lower=-2.6 upper=2.6 effort=100 velocity=2 -> lower=-2.0944 upper=2.0944 effort=108.0 velocity=3.1416; origin xyz=0.12 0 0 rpy=0 0 0 -> xyz=0 0 0 rpy=1.5708 0 0; parent link1_R -> Link1_R
- joint Joint3_L: child link3_L -> Link3_L; limit lower=-2.6 upper=2.6 effort=100 velocity=2 -> lower=-2.9671 upper=2.9671 effort=66.0 velocity=3.1416; origin xyz=0.28 0 0 rpy=0 0 0 -> xyz=0 0.287 0 rpy=-1.5708 0 0; parent link2_L -> Link2_L
- joint Joint3_R: child link3_R -> Link3_R; limit lower=-2.6 upper=2.6 effort=100 velocity=2 -> lower=-2.9671 upper=2.9671 effort=66.0 velocity=3.1416; origin xyz=0.28 0 0 rpy=0 0 0 -> xyz=0 0.287 0 rpy=-1.5708 0 0; parent link2_R -> Link2_R
- joint Joint4_L: child link4_L -> Link4_L; limit lower=-3.0 upper=3.0 effort=100 velocity=2 -> lower=-2.5307 upper=1.0472 effort=66.0 velocity=3.1416; origin xyz=0.25 0 0 rpy=0 0 0 -> xyz=0.018 0 0 rpy=-1.5708 0 3.1416; parent link3_L -> Link3_L
- joint Joint4_R: child link4_R -> Link4_R; limit lower=-3.0 upper=3.0 effort=100 velocity=2 -> lower=-2.5307 upper=1.0472 effort=66.0 velocity=3.1416; origin xyz=0.25 0 0 rpy=0 0 0 -> xyz=0.018 0 0 rpy=-1.5708 0 3.1416; parent link3_R -> Link3_R
- joint Joint5_L: child link5_L -> Link5_L; limit lower=-2.6 upper=2.6 effort=100 velocity=2 -> lower=-2.9671 upper=2.9671 effort=18.0 velocity=3.1416; origin xyz=0.22 0 0 rpy=0 0 0 -> xyz=0.018 -0.314 0 rpy=-1.5708 0 3.1416; parent link4_L -> Link4_L
- joint Joint5_R: child link5_R -> Link5_R; limit lower=-2.6 upper=2.6 effort=100 velocity=2 -> lower=-2.9671 upper=2.9671 effort=18.0 velocity=3.1416; origin xyz=0.22 0 0 rpy=0 0 0 -> xyz=0.018 -0.314 0 rpy=-1.5708 0 3.1416; parent link4_R -> Link4_R
- joint Joint6_L: child link6_L -> Link6_L; limit lower=-3.0 upper=3.0 effort=100 velocity=2 -> lower=-1.0472 upper=1.0472 effort=18.0 velocity=3.1416; origin xyz=0.18 0 0 rpy=0 0 0 -> xyz=0 0 0 rpy=1.5708 -1.5708 0; parent link5_L -> Link5_L
- joint Joint6_R: child link6_R -> Link6_R; limit lower=-3.0 upper=3.0 effort=100 velocity=2 -> lower=-1.0472 upper=1.0472 effort=18.0 velocity=3.1416; origin xyz=0.18 0 0 rpy=0 0 0 -> xyz=0 0 0 rpy=1.5708 -1.5708 0; parent link5_R -> Link5_R
- joint Joint7_L: child flange_L -> Link7_L; limit lower=-3.14159 upper=3.14159 effort=100 velocity=2 -> lower=-1.5708 upper=1.5708 effort=18.0 velocity=3.1416; origin xyz=0.12 0 0 rpy=0 0 0 -> xyz=0 0 0 rpy=1.5708 -1.5708 0; parent link6_L -> Link6_L
- joint Joint7_R: child flange_R -> Link7_R; limit lower=-3.14159 upper=3.14159 effort=100 velocity=2 -> lower=-1.5708 upper=1.5708 effort=18.0 velocity=3.1416; origin xyz=0.12 0 0 rpy=0 0 0 -> xyz=0 0 0 rpy=1.5708 -1.5708 0; parent link6_R -> Link6_R
